File: Power_Stage.kicad_sch (KiCad schematic)
At the start: 36 parts, among them Q1 Q_NMOS_GDS, Q2 Q_NMOS_GDS, Q3 Q_NMOS_GDS, Q4 Q_NMOS_GDS, Q5 Q_NMOS_GDS, Q6 Q_NMOS_GDS

Commit message: Can't remember what these changes are
Parts:
- removed C13, C26, C28: 220nF, Capacitor_SMD:C_0805_2012Metric, symbol Device:C
- removed R11, R12, R16, R19, R20, R28: N.M., Resistor_SMD:R_0603_1608Metric, symbol Device:R
- removed R14, R9: 4mΩ, Resistor_SMD:R_2512_6332Metric, symbol MotorController:TAYLOR_RESISTOR
Connections:
- net GND: now also Q2.3 (S); no longer Q6.3 (S)
- net VSHUNT1P: now also Q6.3 (S); no longer Q2.3 (S)
Other:
- moved on the sheet: NT1, R10
