File: Analog_Sensing.kicad_sch (KiCad schematic)
At the start: 23 parts

Commit message: Can't remember what these changes are
Parts:
- removed C22, C29: N.M, Capacitor_SMD:C_0603_1608Metric, symbol Device:C
Connections:
- net PA0 renamed VBUS_Monitor

Commit message: revision 3
Parts:
- C19, C25: footprint Capacitor_SMD:C_0603_1608Metric -> Capacitor_SMD:C_0402_1005Metric
- R23, R24, R26, R27, R37, R39, R41, R44, R47, R50, R56, R57, R62: footprint Resistor_SMD:R_0603_1608Metric -> Resistor_SMD:R_0402_1005Metric
- R29, R53: footprint Resistor_SMD:R_0603_1608Metric -> Resistor_SMD:R_0402_1005Metric; LCSC (none) -> C409665
Connections:
- net VDDA renamed VDD
